File: Hardware/Qwiic_1x1/SparkFun_Qwiic_UV_Sensor_AS7331.brd (EAGLE design)
At the start: 25.4 x 25.4 mm, 51 parts, among them J1 QWIIC_RA, J2 QWIIC_RA, U1 AS7331

Commit message: v01 ready for review
Parts:
- added U$23: (no value), SparkFun-Aesthetics:ORDERING_INSTRUCTIONS
- U$8: device output:QWIIC_UV_SENSOR0 -> output:SPECTRAL_UV_SENSOR0
- moved FRAME1 5.34 mm to (21.8, -14.2)
- moved U$7 0.28 mm to (6.22, 23.6)
- moved U$25 0.25 mm to (12.7, 7.11)
- moved PWR 0.13 mm to (23.0, 15.5)
- moved U$6 0.13 mm to (23.0, 14.7)
Routing:
- net 3.3V: track 10.3 -> 11.2 mm
Other:
- board text added: "Alex Brudner"
- board text added: "Thickness: 1.6mm Stackup: JLC7628 Layers: 4 Solder Mask Color: Red Silkscreen: White Finish: Lead-Free HASL"
- board text added: "v01"
Changed lines of the file:
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@@
 <layer number="30" name="bStop" color="7" fill="6" visible="yes" active="yes"/>
 <layer number="31" name="tCream" color="7" fill="4" visible="yes" active="yes"/>
-<layer number="32" name="bCream" color="7" fill="5" visible="yes" active="yes"/>
+<layer number="32" name="bCream" color="7" fill="5" visible="no" active="yes"/>
 <layer number="33" name="tFinish" color="6" fill="3" visible="no" active="yes"/>
 <layer number="34" name="bFinish" color="6" fill="6" visible="no" active="yes"/>
@@
 <dimension x1="0" y1="25.4" x2="25.4" y2="25.4" x3="12.7" y3="41.148" textsize="1.27" textratio="15" layer="47" dtype="horizontal" unit="inch"/>
 <text x="4.318" y="44.958" size="1.27" layer="47" ratio="15">All Units in Inches</text>
+<text x="49.149" y="-14.224" size="1.778" layer="51" font="vector" ratio="15">Alex Brudner</text>
+<text x="31.369" y="19.05" size="2.032" layer="51" font="vector">Thickness: 1.6mm
+Stackup: JLC7628
+Layers: 4
+Solder Mask Color: Red
+Silkscreen: White
+Finish: Lead-Free HASL</text>
+<text x="22.098" y="0.254" size="0.889" layer="16" font="vector" ratio="15" rot="MR0">v01</text>
 </plain>
 <attributes>
@@
 </autorouter>
 <elements>
-<element name="FRAME1" library="SparkFun-Aesthetics" package="CREATIVE_COMMONS" value="FRAME-LETTER" x="21.59" y="-8.89" smashed="yes">
-<attribute name="DESIGNER" value="Alex Brudner" x="21.59" y="-8.89" size="1.778" layer="27" display="off"/>
-<attribute name="REV" value="v01" x="21.59" y="-8.89" size="1.778" layer="27" display="off"/>
+<element name="FRAME1" library="SparkFun-Aesthetics" package="CREATIVE_COMMONS" value="FRAME-LETTER" x="21.844" y="-14.224" smashed="yes">
+<attribute name="DESIGNER" value="Alex Brudner" x="21.844" y="-14.224" size="1.778" layer="27" display="off"/>
+<attribute name="REV" value="v01" x="21.844" y="-14.224" size="1.778" layer="27" display="off"/>
 </element>
 <element name="J1" library="SparkFun-Connectors" package="JST04_1MM_RA" value="QWIIC_RA" x="20.32" y="12.7" smashed="yes" rot="R90">
@@
 </element>
 <element name="U1" library="SparkFun_Qwiic_UV_Sensor_AS7331" package="OLGA16" value="AS7331" x="12.7" y="12.7" smashed="yes" rot="R90">
-<attribute name="PROD_ID" value="IC-" x="12.7" y="12.7" size="1.778" layer="27" rot="R90" display="off"/>
+<attribute name="PROD_ID" value="IC-20090" x="12.7" y="12.7" size="1.778" layer="27" rot="R90" display="off"/>
 </element>
 <element name="SUPPLYTIE1" library="SparkFun-PowerSymbols" package="2PT_GND_TIE" value="2PT_GND_TIE" x="10.287" y="14.478" smashed="yes" rot="MR270"/>
@@
 <attribute name="VALUE" x="21.009" y="18.288" size="0.6096" layer="27" font="vector" ratio="20" rot="R90" align="top-center"/>
 </element>
-<element name="PWR" library="SparkFun-Jumpers" package="SMT-JUMPER_2_NC_TRACE_SILK" package3d_urn="urn:adsk.eagle:package:39281/1" value="JUMPER-SMT_2_NC_TRACE_SILK" x="22.86" y="15.494" smashed="yes" rot="MR270">
-<attribute name="NAME" x="21.717" y="15.494" size="0.6096" layer="26" font="vector" ratio="20" rot="MR270" align="bottom-center"/>
-<attribute name="VALUE" x="24.003" y="15.494" size="0.6096" layer="28" font="vector" ratio="20" rot="MR270" align="top-center"/>
+<element name="PWR" library="SparkFun-Jumpers" package="SMT-JUMPER_2_NC_TRACE_SILK" package3d_urn="urn:adsk.eagle:package:39281/1" value="JUMPER-SMT_2_NC_TRACE_SILK" x="22.987" y="15.494" smashed="yes" rot="MR270">
+<attribute name="NAME" x="21.844" y="15.494" size="0.6096" layer="26" font="vector" ratio="20" rot="MR270" align="bottom-center"/>
+<attribute name="VALUE" x="24.13" y="15.494" size="0.6096" layer="28" font="vector" ratio="20" rot="MR270" align="top-center"/>
 </element>
 <element name="R7" library="SparkFun_Qwiic_UV_Sensor_AS7331" package="AXIAL-0.4" value="3.3M" x="12.7" y="21.59" smashed="yes" rot="R180">
 <attribute name="NAME" x="12.827" y="20.574" size="0.6096" layer="25" font="vector" ratio="20" rot="R180" align="bottom-center"/>
 <attribute name="PN" value="MFR-25FTE52-3M3" x="12.827" y="21.59" size="1.778" layer="27" rot="R180" display="off"/>
-<attribute name="PROD_ID" value="RES-" x="12.827" y="21.59" size="1.778" layer="27" rot="R180" display="off"/>
+<attribute name="PROD_ID" value="RES-20091" x="12.827" y="21.59" size="1.778" layer="27" rot="R180" display="off"/>
 <attribute name="VALUE" x="12.7" y="22.606" size="0.6096" layer="27" font="vector" ratio="20" rot="R180" align="top-center"/>
 </element>
@@
 <element name="U$21" library="output" package="#_INT#0" value="" x="16.51" y="1.524" smashed="yes" rot="R90"/>
 <element name="U$22" library="output" package="#_SYN#0" value="" x="19.05" y="1.524" smashed="yes" rot="R90"/>
-<element name="U$6" library="output" package="#PWR#0" value="" x="22.86" y="14.6685" smashed="yes" rot="MR90"/>
+<element name="U$6" library="output" package="#PWR#0" value="" x="22.987" y="14.6685" smashed="yes" rot="MR90"/>
 <element name="U$24" library="output" package="#A1#0" value="" x="4.3815" y="19.05" smashed="yes" rot="MR0"/>
-<element name="U$7" library="SparkFun-Aesthetics" package="SFE_LOGO_FLAME_STOP_.1" value="" x="6.35" y="23.368" smashed="yes"/>
-<element name="U$8" library="output" package="QWIIC_UV_SENSOR0" value="" x="12.7" y="8.89" smashed="yes" rot="MR0"/>
-<element name="U$25" library="output" package="AS73310" value="" x="12.7" y="7.366" smashed="yes" rot="MR0"/>
+<element name="U$7" library="SparkFun-Aesthetics" package="SFE_LOGO_FLAME_STOP_.1" value="" x="6.223" y="23.622" smashed="yes"/>
+<element name="U$25" library="output" package="AS73310" value="" x="12.7" y="7.112" smashed="yes" rot="MR0"/>
 <element name="U$26" library="output" package="#I�C#0" value="" x="2.54" y="9.271" smashed="yes" rot="MR0"/>
 <element name="H3" library="SparkFun-Hardware" package="STAND-OFF-TIGHT" value="STAND-OFFTIGHT" x="2.54" y="22.86" smashed="yes">
@@
 </element>
 <element name="U$9" library="output" package="#A0#0" value="" x="19.685" y="19.05" smashed="yes" rot="MR0"/>
+<element name="U$23" library="SparkFun-Aesthetics" package="ORDERING_INSTRUCTIONS" value="" x="29.464" y="46.355" smashed="yes"/>
+<element name="U$8" library="output" package="SPECTRAL_UV_SENSOR0" value="" x="12.7" y="8.89" smashed="yes" rot="MR0"/>
 </elements>
 <signals>
@@
 <wire x1="16.637" y1="13.843" x2="16.637" y2="13.835" width="0.3048" layer="1"/>
 <via x="16.637" y="13.843" extent="1-16" drill="0.3048"/>
-<via x="21.717" y="14.986" extent="1-16" drill="0.3048"/>
-<wire x1="21.717" y1="14.986" x2="21.7297" y2="14.9733" width="0.3048" layer="16"/>
-<wire x1="21.7297" y1="14.9733" x2="22.86" y2="14.9733" width="0.3048" layer="16"/>
+<via x="21.59" y="16.002" extent="1-16" drill="0.3048"/>
+<wire x1="21.59" y1="16.002" x2="21.59" y2="15.494" width="0.3048" layer="16"/>
+<wire x1="22.1107" y1="14.9733" x2="21.59" y2="15.494" width="0.3048" layer="16"/>
+<wire x1="22.1107" y1="14.9733" x2="22.987" y2="14.9733" width="0.3048" layer="16"/>
 </signal>
 <signal name="VDDA">
-<contactref element="C2" pad="1"/>
-<contactref element="U1" pad="3"/>
 <contactref element="R3" pad="2"/>
 <contactref element="R4" pad="2"/>
-<contactref element="R6" pad="2"/>
-<wire x1="11.15" y1="12.95" x2="11.146" y2="12.946" width="0.3048" layer="1"/>
-<wire x1="11.146" y1="12.946" x2="9.652" y2="12.946" width="0.3048" layer="1"/>
-<wire x1="8.12" y1="12.954" x2="9.644" y2="12.954" width="0.3048" layer="1"/>
-<wire x1="9.644" y1="12.954" x2="9.652" y2="12.946" width="0.3048" layer="1"/>
-<wire x1="9.652" y1="16.01" x2="9.652" y2="12.946" width="0.3048" layer="1"/>
 <wire x1="15.748" y1="15.9846" x2="14.8764" y2="15.9846" width="0.3048" layer="1"/>
 <wire x1="14.8764" y1="15.9846" x2="14.859" y2="16.002" width="0.3048" layer="1"/>
@@
 <wire x1="8.763" y1="16.002" x2="8.771" y2="16.01" width="0.3048" layer="1"/>
 <wire x1="8.771" y1="16.01" x2="9.652" y2="16.01" width="0.3048" layer="1"/>
+<contactref element="C2" pad="1"/>
+<contactref element="U1" pad="3"/>
+<contactref element="R6" pad="2"/>
+<wire x1="11.15" y1="12.95" x2="11.146" y2="12.946" width="0.3048" layer="1"/>
+<wire x1="11.146" y1="12.946" x2="9.652" y2="12.946" width="0.3048" layer="1"/>
+<wire x1="8.12" y1="12.954" x2="9.644" y2="12.954" width="0.3048" layer="1"/>
+<wire x1="9.644" y1="12.954" x2="9.652" y2="12.946" width="0.3048" layer="1"/>
+<wire x1="9.652" y1="12.946" x2="9.652" y2="16.01" width="0.3048" layer="1"/>
 </signal>
 <signal name="N$8">
@@
 <via x="21.463" y="18.796" extent="1-16" drill="0.3048"/>
 <wire x1="21.463" y1="18.796" x2="22.225" y2="18.796" width="0.3048" layer="16"/>
-<wire x1="22.86" y1="18.161" x2="22.86" y2="16.0147" width="0.3048" layer="16"/>
-<wire x1="22.225" y1="18.796" x2="22.86" y2="18.161" width="0.3048" layer="16"/>
+<wire x1="22.987" y1="18.034" x2="22.987" y2="16.0147" width="0.3048" layer="16"/>
+<wire x1="22.225" y1="18.796" x2="22.987" y2="18.034" width="0.3048" layer="16"/>
 </signal>
 </signals>
@@
 </drawing>
 <compatibility>
+<note version="6.3" minversion="6.2.2" severity="warning">
+Since Version 6.2.2 text objects can contain more than one line,
+which will not be processed correctly with this version.
+</note>
 <note version="8.3" severity="warning">
 Since Version 8.3, EAGLE supports URNs for individual library

Commit message: Pushing to v10
Panelize and push to v10.
Parts:
- added U$27: (no value), output:#_#SYN##0
- added U$28: (no value), output:AS73310
- added U$29: (no value), output:SPECTRAL_UV_SENSOR0
- added U$30, U$31: (no value), output:#0#0
- added U$32, U$33: (no value), output:#1#0
- D1: value (none) -> RED; device SparkFun-LED:LED-0603 -> SparkFun-LED:LED-0402
- R5: value 4.7k -> 2.2k
- R7: device SparkFun_Qwiic_UV_Sensor_AS7331:AXIAL-0.4 -> SparkFun_Qwiic_UV_Sensor_AS7331:1206
- U$16: device output:#_SYN#0 -> output:#_#SYN##0
- U$22: device output:#_SYN#0 -> SparkFun-Aesthetics:SFE_LOGO_NAME_.1
- moved U$22 18.0 mm to (12.7, 18.4), turned to 0 degrees
- moved U$24 1.33 mm to (5.71, 19.1)
- moved R7 1.27 mm to (12.7, 22.9)
- moved U$26 1.02 mm to (2.54, 10.3)
- moved I2C 1.02 mm to (2.54, 8.64)
- moved R2 0.46 mm to (1.65, 7.87)
- moved FD1 0.36 mm to (0.89, 24.5)
- moved FD2 0.36 mm to (24.5, 0.89)
- moved FD3 0.36 mm to (0.89, 24.5)
- moved FD4 0.36 mm to (24.5, 0.89)
- moved R1 0.28 mm to (3.68, 7.87)
- moved U$10 0.18 mm to (23.0, 18.9)
- flipped U$16 to the top
- renumbered ADDR0 to A0, ADDR1 to A1
Connections:
- net AGND: now also R7.1; no longer R7.P$1
- net N$8: now also R7.2; no longer R7.P$2
Routing:
- net AGND: track 42.8 -> 45.9 mm
- net N$8: track 9.60 -> 11.8 mm
- net 3.3V: track 11.2 -> 12.2 mm
- net A1: track 15.7 -> 15.2 mm
- net GND: vias 18 -> 17
Other:
- board text added: "1"
- board text added: "2"
- board text added: "3"
- board text added: "4"
- board text added: "Thickness: 1.6mm Stackup: JLC7628 Layers: 4 Copper: 1oz outer, 0.5 oz inner Material: FR-4 TG 135-140 Solder Mask Color: Red Silkscreen: White Finish: Lead-Free HASL"
- board text added: "v10"
- board text removed: "Thickness: 1.6mm Stackup: JLC7628 Layers: 4 Solder Mask Color: Red Silkscreen: White Finish: Lead-Free HASL"
- board text removed: "v01"
