File: Hardware/Qwiic_Mini/SparkFun_Qwiic_Mini_UV_Sensor_AS7331.brd (EAGLE design)
At the start: 25.4 x 12.7 mm, 43 parts, among them J1 Qwiic Vert, J2 Qwiic Vert, U1 AS7331

Commit message: v01 ready for review
Parts:
- added U$19: (no value), SparkFun-Aesthetics:ORDERING_INSTRUCTIONS
- added U$20: (no value), output:SPECTRAL0
- moved U$17 17.9 mm to (21.6, 5.71)
- moved FRAME1 12.8 mm to (21.1, -21.6)
- moved U$18 0.74 mm to (3.43, 6.35)
Other:
- board text added: "Thickness: 1.6mm Stackup: JLC7628 Layers: 4 Solder Mask Color: Red Silkscreen: White Finish: Lead-Free HASL"
- board text added: "v01"
Changed lines of the file:
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@@
 <drawing>
 <settings>
-<setting alwaysvectorfont="no"/>
+<setting alwaysvectorfont="yes"/>
 <setting verticaltext="up"/>
 </settings>
@@
 <wire x1="0" y1="12.7" x2="0" y2="0" width="0.2032" layer="20"/>
 <rectangle x1="16.129" y1="7.747" x2="16.383" y2="7.874" layer="41"/>
-<text x="47.752" y="-8.763" size="1.778" layer="51" font="vector" ratio="15">Alex Brudner</text>
+<text x="48.514" y="-21.59" size="1.778" layer="51" font="vector" ratio="15">Alex Brudner</text>
 <dimension x1="0" y1="0" x2="19.05" y2="1.27" x3="-0.889" y3="0.635" textsize="1.27" layer="47" dtype="vertical" unit="inch"/>
 <dimension x1="0" y1="0" x2="2.54" y2="2.54" x3="-3.175" y3="1.27" textsize="1.27" layer="47" dtype="vertical" unit="inch"/>
@@
 <dimension x1="0" y1="0" x2="25.4" y2="12.7" x3="12.7" y3="28.194" textsize="1.27" layer="47" dtype="horizontal" unit="inch"/>
 <text x="5.334" y="31.623" size="1.27" layer="47" font="vector">All Units in Inches</text>
+<text x="29.21" y="10.541" size="2.032" layer="51" font="vector">Thickness: 1.6mm
+Stackup: JLC7628
+Layers: 4
+Solder Mask Color: Red
+Silkscreen: White
+Finish: Lead-Free HASL</text>
+<text x="22.098" y="0.254" size="0.889" layer="16" font="vector" ratio="15" rot="SMR0">v01</text>
 </plain>
 <attributes>
@@
 </autorouter>
 <elements>
-<element name="FRAME1" library="SparkFun-Aesthetics" package="CREATIVE_COMMONS" value="FRAME-LETTER" x="20.32" y="-8.763" smashed="yes">
-<attribute name="DESIGNER" value="Alex Brudner" x="20.32" y="-8.763" size="1.778" layer="27" display="off"/>
-<attribute name="REV" value="v01" x="20.32" y="-8.763" size="1.778" layer="27" display="off"/>
+<element name="FRAME1" library="SparkFun-Aesthetics" package="CREATIVE_COMMONS" value="FRAME-LETTER" x="21.082" y="-21.59" smashed="yes">
+<attribute name="DESIGNER" value="Alex Brudner" x="21.082" y="-21.59" size="1.778" layer="27" display="off"/>
+<attribute name="REV" value="v01" x="21.082" y="-21.59" size="1.778" layer="27" display="off"/>
 </element>
 <element name="J1" library="SparkFun-Connectors" package="JST04_1MM_VERT" value="Qwiic Vert" x="20.828" y="8.89" smashed="yes" rot="R270">
@@
 </element>
 <element name="U1" library="SparkFun_Qwiic_UV_Sensor_AS7331" package="OLGA16" value="AS7331" x="12.7" y="9.398" smashed="yes" rot="MR90">
-<attribute name="PROD_ID" value="IC-" x="12.7" y="9.398" size="1.778" layer="28" rot="MR90" display="off"/>
+<attribute name="PROD_ID" value="IC-20090" x="12.7" y="9.398" size="1.778" layer="28" rot="MR90" display="off"/>
 </element>
 <element name="SUPPLYTIE1" library="SparkFun-PowerSymbols" package="2PT_GND_TIE" value="2PT_GND_TIE" x="7.747" y="8.763" smashed="yes" rot="MR180"/>
@@
 <attribute name="NAME" x="12.573" y="12.192" size="0.6096" layer="25" font="vector" ratio="20" align="bottom-center"/>
 <attribute name="PN" value="MFR-25FTE52-3M3" x="12.573" y="11.176" size="1.778" layer="27" display="off"/>
-<attribute name="PROD_ID" value="RES-" x="12.573" y="11.176" size="1.778" layer="27" display="off"/>
+<attribute name="PROD_ID" value="RES-20091" x="12.573" y="11.176" size="1.778" layer="27" display="off"/>
 <attribute name="VALUE" x="12.573" y="10.16" size="0.6096" layer="27" font="vector" ratio="20" align="top-center"/>
 </element>
@@
 </element>
 <element name="U$9" library="output" package="#PWR#0" value="" x="16.129" y="4.191" smashed="yes"/>
-<element name="U$17" library="output" package="UV_SENSOR0" value="" x="3.81" y="7.493" smashed="yes" rot="MR0"/>
-<element name="U$18" library="output" package="AS73310" value="" x="3.81" y="5.715" smashed="yes" rot="MR0"/>
+<element name="U$17" library="output" package="UV_SENSOR0" value="" x="21.59" y="5.715" smashed="yes" rot="MR0"/>
+<element name="U$18" library="output" package="AS73310" value="" x="3.429" y="6.35" smashed="yes" rot="MR0"/>
+<element name="U$19" library="SparkFun-Aesthetics" package="ORDERING_INSTRUCTIONS" value="" x="27.559" y="38.227" smashed="yes"/>
+<element name="U$20" library="output" package="SPECTRAL0" value="" x="21.59" y="7.112" smashed="yes" rot="MR0"/>
 </elements>
 <signals>
@@
 </signal>
 <signal name="VDDA">
+<contactref element="R3" pad="2"/>
+<contactref element="R4" pad="2"/>
 <contactref element="C2" pad="1"/>
 <contactref element="U1" pad="3"/>
-<contactref element="R3" pad="2"/>
-<contactref element="R4" pad="2"/>
+<contactref element="R6" pad="2"/>
 <wire x1="14.25" y1="9.648" x2="15.744" y2="9.648" width="0.3048" layer="16"/>
 <wire x1="15.744" y1="9.648" x2="15.748" y2="9.644" width="0.254" layer="16"/>
@@
 <wire x1="12.7" y1="7.366" x2="12.7" y2="6.604" width="0.3048" layer="15"/>
 <via x="12.7" y="6.604" extent="1-16" drill="0.3048"/>
-<contactref element="R6" pad="2"/>
 <wire x1="11.684" y1="5.342" x2="12.684" y2="5.342" width="0.3048" layer="1"/>
 <wire x1="12.684" y1="5.342" x2="12.7" y2="5.326" width="0.3048" layer="1"/>
@@
 </drawing>
 <compatibility>
+<note version="6.3" minversion="6.2.2" severity="warning">
+Since Version 6.2.2 text objects can contain more than one line,
+which will not be processed correctly with this version.
+</note>
 <note version="8.3" severity="warning">
 Since Version 8.3, EAGLE supports URNs for individual library

Commit message: Pushing to v10
Panelize and push to v10.
Parts:
- removed U$16: (no value), output:#_SYN#0
- added U$21: (no value), output:#_#SYN##0
- D1: value (none) -> RED; device SparkFun-LED:LED-0603 -> SparkFun-LED:LED-0402
- R5: value 4.7k -> 2.2k
- R7: device SparkFun_Qwiic_UV_Sensor_AS7331:AXIAL-0.4 -> SparkFun_Qwiic_UV_Sensor_AS7331:1206
- moved FD2 0.36 mm to (24.5, 0.89)
- moved FD4 0.36 mm to (24.5, 0.89)
- moved FD1 0.13 mm to (4.83, 11.9)
- moved FD3 0.13 mm to (4.83, 11.9)
- moved R7 0.13 mm to (12.7, 11.2)
- renumbered ADDR0 to A0, ADDR1 to A1
Connections:
- net SYNC renamed !SYNC
- net AGND: now also R7.1; no longer R7.P$1
- net N$8: now also R7.2; no longer R7.P$2
Routing:
- net !SYNC: track 16.6 -> 23.7 mm
- net READY/INT: track 14.3 -> 18.0 mm
- net N$8: track 4.00 -> 6.04 mm, vias 0 -> 1
- net AGND: track 4.05 -> 4.83 mm, vias 3 -> 2
- net A1: track 4.87 -> 5.42 mm
Other:
- board text added: "1"
- board text added: "2"
- board text added: "3"
- board text added: "4"
- board text added: "Thickness: 1.6mm Stackup: JLC7628 Layers: 4 Copper: 1oz outer, 0.5 oz inner Material: FR-4 TG 135-140 Solder Mask Color: Red Silkscreen: White Finish: Lead-Free HASL"
- board text added: "v10"
- board text removed: "Thickness: 1.6mm Stackup: JLC7628 Layers: 4 Solder Mask Color: Red Silkscreen: White Finish: Lead-Free HASL"
- board text removed: "v01"
