File: Hardware/Qwiic_Mini/SparkFun_Qwiic_Mini_UV_Sensor_AS7331.sch (EAGLE design)
At the start: 30 parts, among them J1 Qwiic Vert, J2 Qwiic Vert, U1 AS7331

Commit message: v01 ready for review
Changed lines of the file:
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@@
 <setting verticaltext="up"/>
 </settings>
-<grid distance="0.1" unitdist="inch" unit="inch" style="lines" multiple="1" display="yes" altdistance="0.05" altunitdist="inch" altunit="inch"/>
+<grid distance="0.1" unitdist="inch" unit="inch" style="lines" multiple="1" display="no" altdistance="0.01" altunitdist="inch" altunit="inch"/>
 <layers>
 <layer number="1" name="Top" color="4" fill="1" visible="no" active="no"/>
@@
 <attribute name="VALUE" x="228.6" y="101.346" size="1.778" layer="96" font="vector" align="top-center"/>
 </instance>
-<instance part="SUPPLY1" gate="G$1" x="63.5" y="139.7" smashed="yes">
-<attribute name="VALUE" x="63.5" y="142.494" size="1.778" layer="96" font="vector" align="bottom-center"/>
+<instance part="SUPPLY1" gate="G$1" x="66.04" y="139.7" smashed="yes">
+<attribute name="VALUE" x="66.04" y="142.494" size="1.778" layer="96" font="vector" align="bottom-center"/>
 </instance>
 <instance part="SUPPLY2" gate="G$1" x="139.7" y="152.4" smashed="yes">
@@
 <net name="VDDA" class="0">
 <segment>
+<pinref part="SUPPLY2" gate="G$1" pin="VDDA"/>
+<pinref part="R3" gate="G$1" pin="2"/>
+<wire x1="139.7" y1="152.4" x2="139.7" y2="149.86" width="0.1524" layer="91"/>
+</segment>
+<segment>
+<pinref part="SUPPLY3" gate="G$1" pin="VDDA"/>
+<pinref part="R4" gate="G$1" pin="2"/>
+<wire x1="152.4" y1="152.4" x2="152.4" y2="149.86" width="0.1524" layer="91"/>
+</segment>
+<segment>
 <pinref part="C2" gate="G$1" pin="1"/>
 <pinref part="U1" gate="G$1" pin="VDDA"/>
 <wire x1="63.5" y1="129.54" x2="63.5" y2="132.08" width="0.1524" layer="91"/>
-<wire x1="63.5" y1="132.08" x2="83.82" y2="132.08" width="0.1524" layer="91"/>
-<pinref part="SUPPLY1" gate="G$1" pin="VDDA"/>
-<wire x1="63.5" y1="139.7" x2="63.5" y2="132.08" width="0.1524" layer="91"/>
+<wire x1="63.5" y1="132.08" x2="66.04" y2="132.08" width="0.1524" layer="91"/>
 <junction x="63.5" y="132.08"/>
 <pinref part="R6" gate="G$1" pin="2"/>
+<wire x1="66.04" y1="132.08" x2="83.82" y2="132.08" width="0.1524" layer="91"/>
 <wire x1="60.96" y1="132.08" x2="63.5" y2="132.08" width="0.1524" layer="91"/>
-</segment>
-<segment>
-<pinref part="SUPPLY2" gate="G$1" pin="VDDA"/>
-<pinref part="R3" gate="G$1" pin="2"/>
-<wire x1="139.7" y1="152.4" x2="139.7" y2="149.86" width="0.1524" layer="91"/>
-</segment>
-<segment>
-<pinref part="SUPPLY3" gate="G$1" pin="VDDA"/>
-<pinref part="R4" gate="G$1" pin="2"/>
-<wire x1="152.4" y1="152.4" x2="152.4" y2="149.86" width="0.1524" layer="91"/>
-</segment>
-</net>
+<pinref part="SUPPLY1" gate="G$1" pin="VDDA"/>
+<wire x1="66.04" y1="139.7" x2="66.04" y2="132.08" width="0.1524" layer="91"/>
+<junction x="66.04" y="132.08"/>
+</segment>
+</net>

Commit message: Pushing to v10
Panelize and push to v10.
Parts:
- D1: value (none) -> RED; device SparkFun-LED:LED-RED_0603-KB -> SparkFun-LED:LED-RED_0402
- FRAME1: REV v01 -> v10
- R5: value 4.7k -> 2.2k; device SparkFun-Resistors:4.7KOHM-0402T-1/16W-1% -> SparkFun-Resistors:2.2KOHM-0402T-1/16W-1%
- renumbered ADDR0 to A0, ADDR1 to A1
Connections:
- net SYNC renamed !SYNC
Other:
- note added: "A0"
- note added: "A1"
- note added: "Cut I2C jumper to remove pull-ups from the I2C lines"
- note added: "Cut and solder A0/A1 pins to change I2C address based on the below table."
- note added: "Voltage Range: 2.7-3.6V"
- note removed: "ADDR0"
- note removed: "ADDR1"
- note removed: "Cut and solder ADDR pins to change I2C address based on the below table."
Changed lines of the file:
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@@
 <part name="FRAME1" library="SparkFun-Aesthetics" deviceset="FRAME-LETTER" device="">
 <attribute name="DESIGNER" value="Alex Brudner"/>
-<attribute name="REV" value="v01"/>
+<attribute name="REV" value="v10"/>
 </part>
 <part name="J1" library="SparkFun-Connectors" deviceset="QWIIC_CONNECTOR" device="" value="Qwiic Vert"/>
@@
 <part name="C1" library="SparkFun-Capacitors" deviceset="0.1UF" device="-0402T-6.3V-10%-X7R" value="0.1uF"/>
 <part name="C2" library="SparkFun-Capacitors" deviceset="0.1UF" device="-0402T-6.3V-10%-X7R" value="0.1uF"/>
-<part name="ADDR0" library="SparkFun-Jumpers" deviceset="JUMPER-SMT_3_1-NC_TRACE" device="_SILK" package3d_urn="urn:adsk.eagle:package:39288/1"/>
-<part name="ADDR1" library="SparkFun-Jumpers" deviceset="JUMPER-SMT_3_1-NC_TRACE" device="_SILK" package3d_urn="urn:adsk.eagle:package:39288/1"/>
+<part name="A0" library="SparkFun-Jumpers" deviceset="JUMPER-SMT_3_1-NC_TRACE" device="_SILK" package3d_urn="urn:adsk.eagle:package:39288/1"/>
+<part name="A1" library="SparkFun-Jumpers" deviceset="JUMPER-SMT_3_1-NC_TRACE" device="_SILK" package3d_urn="urn:adsk.eagle:package:39288/1"/>
 <part name="I2C" library="SparkFun-Jumpers" deviceset="JUMPER-SMT_3_2-NC_TRACE" device="_SILK" package3d_urn="urn:adsk.eagle:package:39289/1"/>
 <part name="R3" library="SparkFun-Resistors" deviceset="10KOHM" device="-0402-1/10W-0.1%" value="10K"/>
@@
 <part name="GND2" library="SparkFun-PowerSymbols" deviceset="DGND" device=""/>
 <part name="GND3" library="SparkFun-PowerSymbols" deviceset="DGND" device=""/>
-<part name="D1" library="SparkFun-LED" deviceset="LED-RED" device="_0603-KB"/>
-<part name="R5" library="SparkFun-Resistors" deviceset="4.7KOHM" device="-0402T-1/16W-1%" value="4.7k"/>
+<part name="D1" library="SparkFun-LED" deviceset="LED-RED" device="_0402" value="RED"/>
+<part name="R5" library="SparkFun-Resistors" deviceset="2.2KOHM" device="-0402T-1/16W-1%" value="2.2k"/>
 <part name="GND4" library="SparkFun-PowerSymbols" deviceset="DGND" device=""/>
 <part name="SUPPLY1" library="SparkFun-PowerSymbols" deviceset="VDDA" device=""/>
@@
 <text x="218.44" y="88.9" size="1.778" layer="97" font="vector">Cut PWR trace to
 disable power LED.</text>
-<text x="157.48" y="119.38" size="1.778" layer="97" font="vector">Cut and solder ADDR
+<text x="157.48" y="119.38" size="1.778" layer="97" font="vector">Cut and solder A0/A1
 pins to change I2C
 address based on the
 below table.</text>
-<text x="172.72" y="91.44" size="1.778" layer="97" font="vector" align="bottom-center">ADDR0</text>
-<text x="160.02" y="91.44" size="1.778" layer="97" font="vector" align="bottom-center">ADDR1</text>
+<text x="172.72" y="91.44" size="1.778" layer="97" font="vector" align="bottom-center">A0</text>
+<text x="160.02" y="91.44" size="1.778" layer="97" font="vector" align="bottom-center">A1</text>
 <text x="190.5" y="91.44" size="1.778" layer="97" font="vector" align="bottom-center">7-bit Address</text>
 <text x="172.72" y="86.36" size="1.778" layer="97" font="vector" align="bottom-center">GND</text>
@@
 <text x="104.14" y="175.26" size="2.54" layer="94" font="vector" align="bottom-center">UV A/B/C Sensor</text>
 <text x="228.6" y="175.26" size="2.54" layer="94" font="vector" align="bottom-center">Power LED</text>
+<text x="129.54" y="162.56" size="1.778" layer="97" font="vector">Cut I2C jumper
+to remove pull-ups
+from the I2C lines</text>
+<text x="96.52" y="147.32" size="1.778" layer="97" font="vector" align="bottom-center">Voltage Range:
+2.7-3.6V</text>
 </plain>
 <instances>
@@
 <attribute name="VALUE" x="65.024" y="122.301" size="1.778" layer="96" font="vector"/>
 </instance>
-<instance part="ADDR0" gate="G$1" x="139.7" y="121.92" smashed="yes">
+<instance part="A0" gate="G$1" x="139.7" y="121.92" smashed="yes">
 <attribute name="NAME" x="142.24" y="121.92" size="1.778" layer="95" font="vector" align="center-left"/>
 </instance>
-<instance part="ADDR1" gate="G$1" x="152.4" y="111.76" smashed="yes">
+<instance part="A1" gate="G$1" x="152.4" y="111.76" smashed="yes">
 <attribute name="NAME" x="154.94" y="111.76" size="1.778" layer="95" font="vector" align="center-left"/>
 </instance>
@@
 <instance part="D1" gate="G$1" x="228.6" y="111.76" smashed="yes">
 <attribute name="NAME" x="231.648" y="112.649" size="1.778" layer="95" font="vector"/>
-<attribute name="VALUE" x="230.505" y="107.188" size="1.778" layer="96" font="vector" rot="R90" align="top-left"/>
+<attribute name="VALUE" x="231.648" y="109.855" size="1.778" layer="96" font="vector" align="top-left"/>
 </instance>
 <instance part="R5" gate="G$1" x="228.6" y="121.92" smashed="yes" rot="R90">
@@
 <segment>
 <pinref part="U1" gate="G$1" pin="A0"/>
-<pinref part="ADDR0" gate="G$1" pin="2"/>
+<pinref part="A0" gate="G$1" pin="2"/>
 <wire x1="109.22" y1="121.92" x2="134.62" y2="121.92" width="0.1524" layer="91"/>
 </segment>
 </net>
-<net name="SYNC" class="0">
+<net name="!SYNC" class="0">
 <segment>
 <pinref part="U1" gate="G$1" pin="SYN"/>
@@
 <segment>
 <pinref part="U1" gate="G$1" pin="A1"/>
-<pinref part="ADDR1" gate="G$1" pin="2"/>
+<pinref part="A1" gate="G$1" pin="2"/>
 <wire x1="109.22" y1="111.76" x2="147.32" y2="111.76" width="0.1524" layer="91"/>
 </segment>
@@
 <net name="N$1" class="0">
 <segment>
-<pinref part="ADDR0" gate="G$1" pin="1"/>
+<pinref part="A0" gate="G$1" pin="1"/>
 <pinref part="R3" gate="G$1" pin="1"/>
 <wire x1="139.7" y1="127" x2="139.7" y2="139.7" width="0.1524" layer="91"/>
@@
 <net name="N$2" class="0">
 <segment>
-<pinref part="ADDR1" gate="G$1" pin="1"/>
+<pinref part="A1" gate="G$1" pin="1"/>
 <pinref part="R4" gate="G$1" pin="1"/>
 <wire x1="152.4" y1="116.84" x2="152.4" y2="139.7" width="0.1524" layer="91"/>
@@
 </segment>
 <segment>
-<pinref part="ADDR1" gate="G$1" pin="3"/>
+<pinref part="A1" gate="G$1" pin="3"/>
 <pinref part="U$1" gate="G$1" pin="AGND"/>
 <wire x1="152.4" y1="106.68" x2="152.4" y2="104.14" width="0.1524" layer="91"/>
 </segment>
 <segment>
-<pinref part="ADDR0" gate="G$1" pin="3"/>
+<pinref part="A0" gate="G$1" pin="3"/>
 <pinref part="U$2" gate="G$1" pin="AGND"/>
 <wire x1="139.7" y1="116.84" x2="139.7" y2="104.14" width="0.1524" layer="91"/>
